Commit message: update monitor_planning_scene

File: excavator_hardware_interface/excavator_description/urdf/sensors/lidar.urdf.xacro (robot description, xacro)
@@ -4,5 +4,5 @@
     <xacro:if value="${'true' == '$(arg use_lidar)' and 'true' == '$(arg use_gazebo)'}">
       <xacro:property name="M_PI" value="3.1415926535897931" />
-      <xacro:property name="lidar_rate" value="50.0"/>
+      <xacro:property name="lidar_rate" value="20.0"/>
       <xacro:property name="lidar_min_dist" value="0.2"/>
       <xacro:property name="lidar_max_dist" value="130.0"/>
@@ -13,5 +13,5 @@
       <xacro:property name="horizontal_resolution" value="0.18"/>
       <xacro:property name="lidar_resolution" value="720"/>
-      <xacro:property name="lidar_channels" value="64"/>
+      <xacro:property name="lidar_channels" value="32"/>
       <link name="lidar_link">
         <inertial>
