Commit message: clock

File: excavator_hardware_interface/excavator_description/urdf/mech/excavator_mech.urdf.xacro (robot description, xacro)
@@ -2,5 +2,5 @@
 <!-- Basic differential drive mobile base -->
 <robot xmlns:xacro="http://www.ros.org/wiki/xacro">
-  <xacro:property name="joint_effort" value="56.0"/>
+  <xacro:property name="joint_effort" value="30.0"/>
   <xacro:property name="joint_velocity" value="2.792527"/>
   <xacro:property name="joint_damping" value="0.0"/>
@@ -11,4 +11,9 @@
   <xacro:property name="arm2_mass" value="0.124"/>
   <xacro:property name="ladle_mass" value="0.11"/>
+  <xacro:property name="wheel_radius" value="0.15"/>
+  <xacro:property name="wheel_width" value="0.1"/>
+  <xacro:property name="wheel_xoff" value="1.08"/>
+  <xacro:property name="wheel_zoff" value="-1.15"/>
+  <xacro:property name="wheel_ygap" value="0.5"/>
   <xacro:macro name="link_inertial" params="mass ixx iyy izz">
     <inertial>
@@ -16,8 +21,47 @@
       <mass value="${mass}"/>
       <inertia
-              ixx="${ixx}" ixy="0.0" ixz="0.0"
-              iyy="${iyy}" iyz="0.0"
-              izz="${izz}"/>
+          ixx="${ixx}" ixy="0.0" ixz="0.0"
+          iyy="${iyy}" iyz="0.0"
+          izz="${izz}"/>
     </inertial>
+  </xacro:macro>
+  <xacro:macro name="cylinder_inertia" params="mass length radius *origin">
+    <inertial>
+      <xacro:insert_block name="origin"/>
+      <mass value="${mass}" />
+      <inertia ixx="${(1/12) * mass * (3*radius*radius + length*length)}" ixy="0.0" ixz="0.0"
+               iyy="${(1/12) * mass * (3*radius*radius + length*length)}" iyz="0.0"
+               izz="${(1/2) * mass * (radius*radius)}" />
+    </inertial>
+  </xacro:macro>
+  <xacro:macro name="wheel" params="prefix x_reflect y_reflect">
+    <link name="${prefix}_link">
+<!--    <visual>-->
+<!--      <origin xyz="0 0 0" rpy="${pi/2} 0 0"/>-->
+<!--      <geometry>-->
+<!--        <cylinder radius="${wheel_radius}" length="${wheel_width}"/>-->
+<!--      </geometry>-->
+<!--      <material name="Gray">-->
+<!--        <color rgba="0.5 0.5 0.5 1.0"/>-->
+<!--      </material>-->
+<!--    </visual>-->
+    <collision>
+      <origin xyz="0 0 0" rpy="${pi/2} 0 0"/>
+      <geometry>
+        <cylinder radius="${wheel_radius}" length="${wheel_width}"/>
+      </geometry>
+    </collision>
+    <xacro:cylinder_inertia mass="0.05" length="${wheel_width}" radius="${wheel_radius}">
+      <origin xyz="0 0 0" rpy="0 0 0"/>
+    </xacro:cylinder_inertia>
+    <!--      <xacro:cylinder_inertia m="0.1" r="${wheel_radius}" h="${wheel_width}"/>-->
+    </link>
+    <joint name="${prefix}_joint" type="revolute">
+      <parent link="base_link"/>
+      <child link="${prefix}_link"/>
+      <origin xyz="${x_reflect*wheel_xoff} ${y_reflect*(1.0/2+wheel_ygap)} ${wheel_zoff}" rpy="0 0 0"/>
+      <axis xyz="0 1 0"/>
+      <limit effort="30" velocity="1.0" lower="-1.79769e+38" upper="1.79769e+38" />
+    </joint>
   </xacro:macro>
   <xacro:macro name="material_visual" params="ref_link ambient diffuse specular">
@@ -35,67 +79,67 @@
     <!-- Robot Base -->
     <link name="base_link">
-      <visual>
-        <geometry>
-          <mesh filename="file://$(find excavator_hardware_interface)/excavator_description/meshes/visual/Down.dae"/>
-        </geometry>
-      </visual>
-      <collision>
-        <geometry>
-          <mesh filename="file://$(find excavator_hardware_interface)/excavator_description/meshes/collision/Down.stl"/>
-        </geometry>
-      </collision>
-      <xacro:link_inertial mass="${base_mass}" ixx="0.000148" iyy="0.000148" izz="0.000096"/>
+    <visual>
+      <geometry>
+        <mesh filename="file://$(find excavator_hardware_interface)/excavator_description/meshes/visual/Down.dae"/>
+      </geometry>
+    </visual>
+    <collision>
+      <geometry>
+        <mesh filename="file://$(find excavator_hardware_interface)/excavator_description/meshes/collision/Down.stl"/>
+      </geometry>
+    </collision>
+    <xacro:link_inertial mass="${base_mass}" ixx="0.000148" iyy="0.000148" izz="0.000096"/>
     </link>
     <link name="cabin_link">
-      <visual>
-        <geometry>
-          <mesh filename="file://$(find excavator_hardware_interface)/excavator_description/meshes/visual/Cabin.dae"/>
-        </geometry>
-      </visual>
-      <collision>
-        <geometry>
-          <mesh filename="file://$(find excavator_hardware_interface)/excavator_description/meshes/collision/Cabin.stl"/>
-        </geometry>
-      </collision>
-      <xacro:link_inertial mass="${cabin_mass}" ixx="0.000148" iyy="0.000148" izz="0.000096"/>
+    <visual>
+      <geometry>
+        <mesh filename="file://$(find excavator_hardware_interface)/excavator_description/meshes/visual/Cabin.dae"/>
+      </geometry>
+    </visual>
+    <collision>
+      <geometry>
+        <mesh filename="file://$(find excavator_hardware_interface)/excavator_description/meshes/collision/Cabin.stl"/>
+      </geometry>
+    </collision>
+    <xacro:link_inertial mass="${cabin_mass}" ixx="0.000148" iyy="0.000148" izz="0.000096"/>
     </link>
     <link name="arm_one_link">
-      <visual>
-        <geometry>
-          <mesh filename="file://$(find excavator_hardware_interface)/excavator_description/meshes/visual/Arm1.dae"/>
-        </geometry>
-      </visual>
-      <collision>
-        <geometry>
-          <mesh filename="file://$(find excavator_hardware_interface)/excavator_description/meshes/collision/Arm1.stl"/>
-        </geometry>
-      </collision>
-      <xacro:link_inertial mass="${arm1_mass}" ixx="0.000148" iyy="0.000148" izz="0.000096"/>
+    <visual>
+      <geometry>
+        <mesh filename="file://$(find excavator_hardware_interface)/excavator_description/meshes/visual/Arm1.dae"/>
+      </geometry>
+    </visual>
+    <collision>
+      <geometry>
+        <mesh filename="file://$(find excavator_hardware_interface)/excavator_description/meshes/collision/Arm1.stl"/>
+      </geometry>
+    </collision>
+    <xacro:link_inertial mass="${arm1_mass}" ixx="0.000148" iyy="0.000148" izz="0.000096"/>
     </link>
     <link name="arm_two_link">
-      <visual>
-        <geometry>
-          <mesh filename="file://$(find excavator_hardware_interface)/excavator_description/meshes/visual/Arm2.dae"/>
-        </geometry>
-      </visual>
-      <collision>
-        <geometry>
-          <mesh filename="file://$(find excavator_hardware_interface)/excavator_description/meshes/collision/Arm2.stl"/>
-        </geometry>
-      </collision>
-      <xacro:link_inertial mass="${arm2_mass}" ixx="0.000148" iyy="0.000148" izz="0.000096"/>
+    <visual>
+      <geometry>
+        <mesh filename="file://$(find excavator_hardware_interface)/excavator_description/meshes/visual/Arm2.dae"/>
+      </geometry>
+    </visual>
+    <collision>
+      <geometry>
+        <mesh filename="file://$(find excavator_hardware_interface)/excavator_description/meshes/collision/Arm2.stl"/>
+      </geometry>
+    </collision>
+    <xacro:link_inertial mass="${arm2_mass}" ixx="0.000148" iyy="0.000148" izz="0.000096"/>
     </link>
     <link name="ladle_link">
-      <visual>
-        <geometry>
-          <mesh filename="file://$(find excavator_hardware_interface)/excavator_description/meshes/visual/Ladle2.dae"/>
-        </geometry>
-      </visual>
-      <collision>
-        <geometry>
-          <mesh filename="file://$(find excavator_hardware_interface)/excavator_description/meshes/collision/Ladle2.stl"/>
-        </geometry>
-      </collision>
-      <xacro:link_inertial mass="${ladle_mass}" ixx="0.000148" iyy="0.000148" izz="0.000096"/>
+    <visual>
+      <geometry>
+        <mesh filename="file://$(find excavator_hardware_interface)/excavator_description/meshes/visual/Ladle2.dae"/>
+      </geometry>
+    </visual>
+    <collision>
+      <geometry>
+        <mesh filename="file://$(find excavator_hardware_interface)/excavator_description/meshes/collision/Ladle2.stl"/>
+      </geometry>
+    </collision>
+    <xacro:link_inertial mass="${ladle_mass}" ixx="0.000148" iyy="0.000148" izz="0.000096"/>
     </link>
     <joint name="cabin_joint" type="revolute">
@@ -104,4 +148,5 @@
       <origin xyz="0.0 0.0 0.0" rpy="0 0 0"/>
       <limit effort="${joint_effort}" lower="-1.56" upper="1.56" velocity="${joint_velocity}"/>
+      <dynamics damping="${joint_damping}" friction="${joint_friction}"/>
       <axis xyz="0 0 1"/>
     </joint>
@@ -110,5 +155,5 @@
       <child link="arm_one_link"/>
       <origin xyz="0.95 -0.17 -0.28" rpy="0 0 0"/>
-      <limit effort="${joint_effort}" lower="-1.6" upper="0.0" velocity="${joint_velocity}"/>
+      <limit effort="${joint_effort}" lower="-1.6" upper="0.0001" velocity="${joint_velocity}"/>
       <dynamics damping="${joint_damping}" friction="${joint_friction}"/>
       <axis xyz="0 1 0"/>
@@ -118,5 +163,5 @@
       <child link="arm_two_link"/>
       <origin xyz="2.66 0.0 -0.62" rpy="0 0 0"/>
-      <limit effort="${joint_effort}" lower="-1.6" upper="0.0" velocity="${joint_velocity}"/>
+      <limit effort="${joint_effort}" lower="-1.6" upper="0.0001" velocity="${joint_velocity}"/>
       <dynamics damping="${joint_damping}" friction="${joint_friction}"/>
       <axis xyz="0 1 0"/>
@@ -126,5 +171,5 @@
       <child link="ladle_link"/>
       <origin xyz="-1.755 0.0 -0.065" rpy="0 0 0"/>
-      <limit effort="${joint_effort}" lower="-1.6" upper="0.0" velocity="${joint_velocity}"/>
+      <limit effort="${joint_effort}" lower="-1.6" upper="0.0001" velocity="${joint_velocity}"/>
       <dynamics damping="${joint_damping}" friction="${joint_friction}"/>
       <axis xyz="0 1 0"/>
@@ -141,4 +186,41 @@
     <xacro:material_visual ref_link="arm2_link" ambient="1 1 1 1" diffuse="1 1 1 1" specular="1 1 1 1"/>
     <xacro:material_visual ref_link="ladle_link" ambient="1 1 1 1" diffuse="1 1 1 1" specular="1 1 1 1"/>
+<!--    <xacro:wheel prefix="wheel_front_left" x_reflect="1" y_reflect="1"/>-->
+<!--    <xacro:wheel prefix="wheel_rear_left" x_reflect="-1" y_reflect="1"/>-->
+<!--    <xacro:wheel prefix="wheel_front_right" x_reflect="1" y_reflect="-1"/>-->
+<!--    <xacro:wheel prefix="wheel_rear_right" x_reflect="-1" y_reflect="-1"/>-->
+<!--    <gazebo>-->
+<!--      <plugin-->
+<!--          filename="gz-sim-diff-drive-system"-->
+<!--          name="gz::sim::systems::DiffDrive">-->
+<!--        <left_joint>wheel_front_left_joint</left_joint>-->
+<!--        <left_joint>wheel_rear_left_joint</left_joint>-->
+<!--        <right_joint>wheel_front_right_joint</right_joint>-->
+<!--        <right_joint>wheel_rear_right_joint</right_joint>-->
+<!--        <wheel_separation>2.05</wheel_separation>-->
+<!--        <wheel_radius>0.15</wheel_radius>-->
+<!--        &lt;!&ndash;    <min_velocity>0.0</min_velocity>&ndash;&gt;-->
+<!--        &lt;!&ndash;    <max_velocity>5.0</max_velocity>&ndash;&gt;-->
+<!--        &lt;!&ndash;    <min_acceleration>0.0</min_acceleration>&ndash;&gt;-->
+<!--        &lt;!&ndash;    <max_acceleration>1.0</max_acceleration>&ndash;&gt;-->
+<!--        &lt;!&ndash;    <min_jerk>1.0</min_jerk>&ndash;&gt;-->
+<!--        &lt;!&ndash;    <max_jerk>3.0</max_jerk>&ndash;&gt;-->
+<!--        <odom_publish_frequency>10</odom_publish_frequency>-->
+<!--        <topic>cmd_vel</topic>-->
+<!--        <odom_topic>odom</odom_topic>-->
+<!--        <tf_topic>/tf</tf_topic>-->
+<!--        <frame_id>odom</frame_id>-->
+<!--        <child_frame_id>base_link</child_frame_id>-->
+<!--      </plugin>-->
+<!--&lt;!&ndash;      <plugin filename="gz-sim-joint-state-publisher-system"&ndash;&gt;-->
+<!--&lt;!&ndash;              name="gz::sim::systems::JointStatePublisher">&ndash;&gt;-->
+<!--&lt;!&ndash;        <topic>joint_states</topic>&ndash;&gt;-->
+<!--&lt;!&ndash;        <joint_name>wheel_front_left_joint</joint_name>&ndash;&gt;-->
+<!--&lt;!&ndash;        <joint_name>wheel_rear_left_joint</joint_name>&ndash;&gt;-->
+<!--&lt;!&ndash;        <joint_name>wheel_front_right_joint</joint_name>&ndash;&gt;-->
+<!--&lt;!&ndash;        <joint_name>wheel_rear_right_joint</joint_name>&ndash;&gt;-->
+<!--&lt;!&ndash;        <joint_name>base_joint</joint_name>&ndash;&gt;-->
+<!--&lt;!&ndash;      </plugin>&ndash;&gt;-->
+<!--    </gazebo>-->
   </xacro:macro>
 </robot>

File: excavator_hardware_interface/excavator_description/urdf/robot/excavator.urdf.xacro (robot description, xacro)
@@ -5,12 +5,12 @@
     <xacro:arg name="use_lidar" default="false"/>
     <xacro:arg name="use_gazebo" default="false"/>
-    <xacro:if value="$(arg add_world)">
-        <link name="world"/>
-        <joint name="virtual_joint" type="fixed">
-            <parent link="world"/>
-            <child link="$(arg base_link)"/>
-            <origin xyz="0 0 0" rpy="0 0 0"/>
-        </joint>
-    </xacro:if>
+<!--    <xacro:if value="$(arg add_world)">-->
+<!--        <link name="base_footprint"/>-->
+<!--        <joint name="base_joint" type="fixed">-->
+<!--            <parent link="base_footprint"/>-->
+<!--            <child link="$(arg base_link)"/>-->
+<!--            <origin xyz="0 0 0" rpy="0 0 0"/>-->
+<!--        </joint>-->
+<!--    </xacro:if>-->
     <xacro:include filename="$(find excavator_hardware_interface)/excavator_description/urdf/mech/excavator_mech.urdf.xacro"/>
     <xacro:excavator

File: excavator_hardware_interface/excavator_description/urdf/sensors/lidar.urdf.xacro (robot description, xacro)
@@ -41,5 +41,5 @@
         <sensor type="gpu_lidar" name="ouster_lidar">
           <pose>0 0 0 0 0 0</pose>
-          <ray>
+          <lidar>
             <scan>
               <horizontal>
@@ -61,10 +61,5 @@
               <resolution>0.001</resolution>
             </range>
-<!--            <noise>-->
-<!--              <type>gaussian</type>-->
-<!--              <mean>${mean}</mean>-->
-<!--              <stddev>${stddev}</stddev>-->
-<!--            </noise>-->
-          </ray>
+          </lidar>
           <update_rate>${lidar_rate}</update_rate>
           <always_on>1</always_on>

Commit message: Done joint

File: excavator_hardware_interface/excavator_description/urdf/mech/excavator_mech.urdf.xacro (robot description, xacro)
@@ -6,5 +6,5 @@
   <xacro:property name="joint_damping" value="0.0"/>
   <xacro:property name="joint_friction" value="0.0"/>
-  <xacro:property name="base_mass" value="0.12"/>
+  <xacro:property name="base_mass" value="10.12"/>
   <xacro:property name="cabin_mass" value="0.19"/>
   <xacro:property name="arm1_mass" value="0.16"/>
@@ -190,5 +190,5 @@
 <!--    <xacro:wheel prefix="wheel_front_right" x_reflect="1" y_reflect="-1"/>-->
 <!--    <xacro:wheel prefix="wheel_rear_right" x_reflect="-1" y_reflect="-1"/>-->
-<!--    <gazebo>-->
+    <gazebo>
 <!--      <plugin-->
 <!--          filename="gz-sim-diff-drive-system"-->
@@ -213,14 +213,15 @@
 <!--        <child_frame_id>base_link</child_frame_id>-->
 <!--      </plugin>-->
-<!--&lt;!&ndash;      <plugin filename="gz-sim-joint-state-publisher-system"&ndash;&gt;-->
-<!--&lt;!&ndash;              name="gz::sim::systems::JointStatePublisher">&ndash;&gt;-->
-<!--&lt;!&ndash;        <topic>joint_states</topic>&ndash;&gt;-->
-<!--&lt;!&ndash;        <joint_name>wheel_front_left_joint</joint_name>&ndash;&gt;-->
-<!--&lt;!&ndash;        <joint_name>wheel_rear_left_joint</joint_name>&ndash;&gt;-->
-<!--&lt;!&ndash;        <joint_name>wheel_front_right_joint</joint_name>&ndash;&gt;-->
-<!--&lt;!&ndash;        <joint_name>wheel_rear_right_joint</joint_name>&ndash;&gt;-->
-<!--&lt;!&ndash;        <joint_name>base_joint</joint_name>&ndash;&gt;-->
-<!--&lt;!&ndash;      </plugin>&ndash;&gt;-->
-<!--    </gazebo>-->
+      <plugin filename="gz-sim-joint-state-publisher-system"
+              name="gz::sim::systems::JointStatePublisher">
+        <topic>joint_states</topic>
+        <joint_name>tool0</joint_name>
+        <joint_name>ladle_link</joint_name>
+        <joint_name>arm_two_link</joint_name>
+        <joint_name>arm_one_link</joint_name>
+        <joint_name>cabin_link</joint_name>
+        <joint_name>base_joint</joint_name>
+      </plugin>
+    </gazebo>
   </xacro:macro>
 </robot>

File: excavator_hardware_interface/excavator_description/urdf/sensors/lidar.urdf.xacro (robot description, xacro)
@@ -4,5 +4,5 @@
     <xacro:if value="${'true' == '$(arg use_lidar)' and 'true' == '$(arg use_gazebo)'}">
       <xacro:property name="M_PI" value="3.1415926535897931" />
-      <xacro:property name="lidar_rate" value="10.0"/>
+      <xacro:property name="lidar_rate" value="50.0"/>
       <xacro:property name="lidar_min_dist" value="0.2"/>
       <xacro:property name="lidar_max_dist" value="130.0"/>

Commit message: Visualization Excavator

File: excavator_hardware_interface/excavator_description/urdf/mech/excavator_mech.urdf.xacro (robot description, xacro)
@@ -146,5 +146,5 @@
       <parent link="base_link"/>
       <child link="cabin_link"/>
-      <origin xyz="0.0 0.0 0.0" rpy="0 0 0"/>
+      <origin xyz="0.0 0.0 1.3" rpy="0 0 0"/>
       <limit effort="${joint_effort}" lower="-1.56" upper="1.56" velocity="${joint_velocity}"/>
       <dynamics damping="${joint_damping}" friction="${joint_friction}"/>
